Commit message: Basic Functionality Restored

File: description/gazebo_control.xacro (robot description, xacro)
@@ -3,10 +3,6 @@
     <gazebo>
         <plugin name="diff_drive" filename="libgazebo_ros_diff_drive.so">
-            <!-- Wheel Information -->
-            <num_wheel_pairs>2</num_wheel_pairs>
-            <left_joint>back_left_wheel_joint</left_joint>
-            <left_joint>front_left_wheel_joint</left_joint>
-            <right_joint>back_right_wheel_joint</right_joint>
-            <right_joint>front_right_wheel_joint</right_joint>
+            <left_joint>left_wheel_joint</left_joint>
+            <right_joint>right_wheel_joint</right_joint>
             <wheel_separation>0.2286</wheel_separation>
             <wheel_diameter>0.1524</wheel_diameter>

File: description/robot.urdf.xacro (robot description, xacro)
@@ -2,10 +2,5 @@
 <robot xmlns:xacro="http://www.ros.org/wiki/xacro"  name="robot">
     <xacro:arg name="use_ros2_control" default="true"/>
-    <!-- <xacro:if value="$(arg sim_mode)"> -->
-        <!-- <xacro:include filename="robot_core_sim.xacro" /> -->
-    <!-- </xacro:if>
-    <xacro:unless value="$(arg sim_mode)"> -->
-        <xacro:include filename="robot_core_hw.xacro" />
-    <!-- </xacro:unless> -->
+    <xacro:include filename="robot_core.xacro" />
     <xacro:if value="$(arg use_ros2_control)">
         <xacro:include filename="ros2_control.xacro" />

File: description/robot_core.xacro (robot description, xacro)
@@ -11,11 +11,11 @@
     <xacro:property name="chassis_top_mass" value="1.0"/>
     <xacro:property name="lid_thickness" value="0.0254"/>
-    <xacro:property name="wheel_radius" value="0.0762"/>
+    <xacro:property name="wheel_radius" value="0.0635"/>
     <xacro:property name="wheel_thickness" value="0.0254"/>
     <xacro:property name="wheel_mass" value="0.05"/>
-    <xacro:property name="front_wheel_offset_x" value="0.22733"/>
-    <xacro:property name="back_wheel_offset_x" value="0.291465"/>
     <xacro:property name="wheel_offset_y" value="0.1143"/>
     <xacro:property name="wheel_offset_z" value="0.026035"/>
+    <xacro:property name="front_caster_wheel_offset_x" value="0.127"/>
+    <xacro:property name="back_caster_wheel_offset_x" value="-0.127"/>
     <material name="white">
         <color rgba="1 1 1 1" />
@@ -54,5 +54,5 @@
         <parent link="base_link"/>
         <child link="chassis_base"/>
-        <origin xyz="${-back_wheel_offset_x} 0 ${-wheel_offset_z}"/>
+        <origin xyz="${-chassis_base_length/2} 0 ${-wheel_offset_z}"/>
     </joint>
     <link name="chassis_base">
@@ -126,12 +126,12 @@
         <material>Gazebo/Black</material>
     </gazebo>
-    <!-- FRONT LEFT WHEEL LINK -->
-    <joint name="front_left_wheel_joint" type="continuous">
-        <parent link="base_link"/>
-        <child link="front_left_wheel"/>
+    <!-- LEFT WHEEL LINK -->
+    <joint name="left_wheel_joint" type="continuous">
+        <parent link="base_link"/>
+        <child link="left_wheel"/>
         <origin xyz="0 ${wheel_offset_y} 0" rpy="-${pi/2} 0 0" />
         <axis xyz="0 0 1"/>
     </joint>
-    <link name="front_left_wheel">
+    <link name="left_wheel">
         <visual>
             <geometry>
@@ -150,19 +150,19 @@
         </xacro:inertial_cylinder>
     </link>
-    <gazebo reference="front_left_wheel">
+    <gazebo reference="left_wheel">
         <material>Gazebo/Gray</material>
     </gazebo>
-    <!-- BACK LEFT WHEEL LINK -->
-    <joint name="back_left_wheel_joint" type="continuous">
-        <parent link="base_link"/>
-        <child link="back_left_wheel"/>
-        <origin xyz="${-front_wheel_offset_x} ${wheel_offset_y} 0" rpy="-${pi/2} 0 0" />
-        <axis xyz="0 0 1"/>
-    </joint>
-    <link name="back_left_wheel">
+    <!-- RIGHT WHEEL LINK -->
+    <joint name="right_wheel_joint" type="continuous">
+        <parent link="base_link"/>
+        <child link="right_wheel"/>
+        <origin xyz="0 ${-wheel_offset_y} 0" rpy="${pi/2} 0 0" />
+        <axis xyz="0 0 -1"/>
+    </joint>
+    <link name="right_wheel">
         <visual>
             <geometry>
                 <cylinder radius="${wheel_radius}" length="${wheel_thickness}"/>
-            </geometry>
+            </geometry>-
             <material name="gray"/>
         </visual>
@@ -177,60 +177,60 @@
         </xacro:inertial_cylinder>
     </link>
-    <gazebo reference="back_left_wheel">
+    <gazebo reference="right_wheel">
         <material>Gazebo/Gray</material>
     </gazebo>
-    <!-- FRONT RIGHT WHEEL LINK -->
-    <joint name="front_right_wheel_joint" type="continuous">
-        <parent link="base_link"/>
-        <child link="front_right_wheel"/>
-        <origin xyz="0 ${-wheel_offset_y} 0" rpy="${pi/2} 0 0" />
-        <axis xyz="0 0 -1"/>
-    </joint>
-    <link name="front_right_wheel">
-        <visual>
-            <geometry>
-                <cylinder radius="${wheel_radius}" length="${wheel_thickness}"/>
-            </geometry>
-            <material name="gray"/>
-        </visual>
-        <collision>
-            <geometry>
-                <sphere radius="${wheel_radius}"/>
-            </geometry>
-        </collision>
-        <xacro:inertial_cylinder mass="${wheel_mass}" length="${wheel_thickness}" radius="${wheel_radius}">
-            <!-- origin should match visual origin -->
-            <origin xyz="0 0 0" rpy="0 0 0"/>
-        </xacro:inertial_cylinder>
-    </link>
-    <gazebo reference="front_right_wheel">
-        <material>Gazebo/Gray</material>
-    </gazebo>
-    <!-- BACK RIGHT WHEEL LINK -->
-    <joint name="back_right_wheel_joint" type="continuous">
-        <parent link="base_link"/>
-        <child link="back_right_wheel"/>
-        <origin xyz="${-front_wheel_offset_x} ${-wheel_offset_y} 0" rpy="${pi/2} 0 0" />
-        <axis xyz="0 0 -1"/>
-    </joint>
-    <link name="back_right_wheel">
-        <visual>
-            <geometry>
-                <cylinder radius="${wheel_radius}" length="${wheel_thickness}"/>
-            </geometry>
-            <material name="gray"/>
-        </visual>
-        <collision>
-            <geometry>
-                <sphere radius="${wheel_radius}"/>
-            </geometry>
-        </collision>
-        <xacro:inertial_cylinder mass="${wheel_mass}" length="${wheel_thickness}" radius="${wheel_radius}">
-            <!-- origin should match visual origin -->
-            <origin xyz="0 0 0" rpy="0 0 0"/>
-        </xacro:inertial_cylinder>
-    </link>
-    <gazebo reference="back_right_wheel">
-        <material>Gazebo/Gray</material>
+    <!-- FRONT CASTER WHEEL LINK -->
+    <joint name="front_caster_wheel_joint" type="fixed">
+        <parent link="base_link"/>
+        <child link="front_caster_wheel"/>
+        <origin xyz="${front_caster_wheel_offset_x} 0 0"/>
+    </joint>
+    <link name="front_caster_wheel">
+        <visual>
+            <geometry>
+                <sphere radius="${wheel_radius}"/>
+            </geometry>
+            <material name="white"/>
+        </visual>
+        <collision>
+            <geometry>
+                <sphere radius="${wheel_radius}"/>
+            </geometry>
+        </collision>
+        <xacro:inertial_sphere mass="${wheel_mass}" radius="${wheel_radius}">
+            <origin xyz="0 0 0" rpy="0 0 0"/>
+        </xacro:inertial_sphere>
+    </link>
+    <gazebo reference="front_caster_wheel">
+        <material>Gazebo/White</material>
+        <mu1 value="0.001"/>
+        <mu2 value="0.001"/>
+    </gazebo>
+    <!-- BACK CASTER WHEEL LINK -->
+    <joint name="back_caster_wheel_joint" type="fixed">
+        <parent link="base_link"/>
+        <child link="back_caster_wheel"/>
+        <origin xyz="${back_caster_wheel_offset_x} 0 0"/>
+    </joint>
+    <link name="back_caster_wheel">
+        <visual>
+            <geometry>
+                <sphere radius="${wheel_radius}"/>
+            </geometry>
+            <material name="white"/>
+        </visual>
+        <collision>
+            <geometry>
+                <sphere radius="${wheel_radius}"/>
+            </geometry>
+        </collision>
+        <xacro:inertial_sphere mass="${wheel_mass}" radius="${wheel_radius}">
+            <origin xyz="0 0 0" rpy="0 0 0"/>
+        </xacro:inertial_sphere>
+    </link>
+    <gazebo reference="back_caster_wheel">
+        <material>Gazebo/White</material>
+        <mu1 value="0.001"/>
+        <mu2 value="0.001"/>
     </gazebo>
 </robot>

File: description/ros2_control.xacro (robot description, xacro)
@@ -36,5 +36,5 @@
                 <plugin>gazebo_ros2_control/GazeboSystem</plugin>
             </hardware>
-            <joint name="front_left_wheel_joint">
+            <joint name="left_wheel_joint">
                 <command_interface name="velocity">
                     <param name="min">-10</param>
@@ -44,21 +44,5 @@
                 <state_interface name="velocity" />
             </joint>
-            <joint name="back_left_wheel_joint">
-                <command_interface name="velocity">
-                    <param name="min">-10</param>
-                    <param name="max">10</param>
-                </command_interface>
-                <state_interface name="position" />
-                <state_interface name="velocity" />
-            </joint>
-            <joint name="front_right_wheel_joint">
-                <command_interface name="velocity">
-                    <param name="min">-10</param>
-                    <param name="max">10</param>
-                </command_interface>
-                <state_interface name="velocity" />
-                <state_interface name="position" />
-            </joint>
-            <joint name="back_right_wheel_joint">
+            <joint name="right_wheel_joint">
                 <command_interface name="velocity">
                     <param name="min">-10</param>
